Commit message: add pd setpoint control

File: fer_drake.urdf (robot description, URDF)
Before this commit: robot fer, 14 links, 13 joints
Links:
- link fer_hand: geometry collision mesh filename=package://franka_description/meshes/robot_ee/franka_hand_wh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; visual mesh filename=package://franka_description/meshes/robot_ee/franka_hand_wh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
- link fer_link0: geometry collision mesh filename=package://franka_description/meshes/robot_arms/fer/collisio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; visual mesh filename=package://franka_description/meshes/robot_arms/fer/visual/l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
- link fer_link1: geometry collision mesh filename=package://franka_description/meshes/robot_arms/fer/collisio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; visual mesh filename=package://franka_description/meshes/robot_arms/fer/visual/l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
- link fer_link2: geometry collision mesh filename=package://franka_description/meshes/robot_arms/fer/collisio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; visual mesh filename=package://franka_description/meshes/robot_arms/fer/visual/l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
- link fer_link3: geometry collision mesh filename=package://franka_description/meshes/robot_arms/fer/collisio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; visual mesh filename=package://franka_description/meshes/robot_arms/fer/visual/l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
- link fer_link4: geometry collision mesh filename=package://franka_description/meshes/robot_arms/fer/collisio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; visual mesh filename=package://franka_description/meshes/robot_arms/fer/visual/l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
- link fer_link5: geometry collision mesh filename=package://franka_description/meshes/robot_arms/fer/collisio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; visual mesh filename=package://franka_description/meshes/robot_arms/fer/visual/l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
- link fer_link6: geometry collision mesh filename=package://franka_description/meshes/robot_arms/fer/collisio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; visual mesh filename=package://franka_description/meshes/robot_arms/fer/visual/l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
- link fer_link7: geometry collision mesh filename=package://franka_description/meshes/robot_arms/fer/collisio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; visual mesh filename=package://franka_description/meshes/robot_arms/fer/visual/l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

Commit message: Configure time step as a CLI argument and add a small PID control component

File: fer_drake.urdf (robot description, URDF)
Before this commit: robot fer, 14 links, 13 joints
Links:
- link fer_leftfinger: mass None -> 0.01
- link fer_rightfinger: mass None -> 0.01
