Commit message: Remove j7

File: fer_drake_fingerless.urdf (robot description, URDF)
Before this commit: robot fer, 9 links, 8 joints
Joints:
- removed joint fer_joint7

Commit message: Setup a franka without joint 7

File: fer_drake_fingerless.urdf (robot description, URDF)
Before this commit: robot fer, 9 links, 7 joints
Links:
- removed link fer_link7

Commit message: Add last joint as fixed

File: fer_drake_fingerless.urdf (robot description, URDF)
Before this commit: robot fer, 9 links, 8 joints
Joints:
- joint fer_joint7: axis 0 0 1 -> (none); limit lower=-2.8973 upper=2.8973 effort=25.0 velocity=2.61 -> (none); type revolute -> fixed

Commit message: g comp works

File: fer_drake_fingerless.urdf (robot description, URDF)
Before this commit: robot fer, 9 links, 8 joints
Joints:
- joint fer_joint7: axis (none) -> 0 0 1; limit (none) -> lower=-2.8973 upper=2.8973 effort=12.0 velocity=2.61; type fixed -> revolute
