Commit message: Add dae models to main repo

File: models/urdf/fer_drake_fingerless.urdf (robot description, URDF)
Before this commit: robot fer, 9 links, 8 joints
Links:
- link fer_link0: geometry collision mesh filename=../meshes/robot_arms/fer/collision/link0.obj; visual mesh filename=../meshes/robot_arms/fer/visual/link0.dae
- link fer_link1: geometry collision mesh filename=../meshes/robot_arms/fer/collision/link1.obj; visual mesh filename=../meshes/robot_arms/fer/visual/link1.dae
- link fer_link2: geometry collision mesh filename=../meshes/robot_arms/fer/collision/link2.obj; visual mesh filename=../meshes/robot_arms/fer/visual/link2.dae
- link fer_link3: geometry collision mesh filename=../meshes/robot_arms/fer/collision/link3.obj; visual mesh filename=../meshes/robot_arms/fer/visual/link3.dae
- link fer_link4: geometry collision mesh filename=../meshes/robot_arms/fer/collision/link4.obj; visual mesh filename=../meshes/robot_arms/fer/visual/link4.dae
- link fer_link5: geometry collision mesh filename=../meshes/robot_arms/fer/collision/link5.obj; visual mesh filename=../meshes/robot_arms/fer/visual/link5.dae
- link fer_link6: geometry collision mesh filename=../meshes/robot_arms/fer/collision/link6.obj; visual mesh filename=../meshes/robot_arms/fer/visual/link6.dae
- link fer_link7: geometry collision mesh filename=../meshes/robot_arms/fer/collision/link7.obj; visual mesh filename=../meshes/robot_arms/fer/visual/link7.dae
