Commit message: Improve urdf collisions

File: models/urdf/fer_drake_gripper_fixed.urdf (robot description, URDF)
Before this commit: robot fer, 14 links, 13 joints
Links:
- link fer_hand: geometry visual mesh filename=../meshes/robot_ee/franka_hand_white/visual/hand.dae
- link fer_leftfinger: geometry collision box size=16e-3 12e-3 10e-3; collision box size=16e-3 7e-3 44e-3
- link fer_rightfinger: geometry collision box size=16e-3 12e-3 10e-3; collision box size=16e-3 7e-3 44e-3

Commit message: Improve gripper

File: models/urdf/fer_drake_gripper_fixed.urdf (robot description, URDF)
Before this commit: robot fer, 14 links, 13 joints
Links:
- link fer_leftfinger: geometry collision box size=14e-3 10e-3 10e-3; collision box size=16e-3 7e-3 44e-3
- link fer_rightfinger: geometry collision box size=14e-3 10e-3 10e-3; collision box size=16e-3 7e-3 44e-3
Joints:
- joint fer_finger_joint1: limit lower=0.0 upper=0.04 effort=100 velocity=0.2 -> lower=0.0 upper=0.04 effort=150 velocity=0.25
- joint fer_finger_joint2: limit lower=0.0 upper=0.04 effort=100 velocity=0.2 -> lower=0.0 upper=0.04 effort=150 velocity=0.25
