Commit message: Collisions fixed

File: models/urdf/fer_drake_gripper_simple_collision.urdf (robot description, URDF)
Before this commit: robot fer, 14 links, 13 joints
Links:
- link fer_hand: geometry collision box size=0.04 0.03 0.03; visual mesh filename=../meshes/robot_ee/franka_hand_white/visual/hand.dae
- link fer_leftfinger: geometry collision box size=0.008 0.012 0.035; visual mesh filename=../meshes/robot_ee/franka_hand_white/visual/finger.dae
- link fer_link0: geometry collision cylinder length=0.2 radius=0.06; visual mesh filename=../meshes/robot_arms/fer/visual/link0.dae
- link fer_link1: geometry collision cylinder length=0.1 radius=0.05; visual mesh filename=../meshes/robot_arms/fer/visual/link1.dae
- link fer_link2: geometry collision box size=0.08 0.2 0.08; visual mesh filename=../meshes/robot_arms/fer/visual/link2.dae
- link fer_link3: geometry collision box size=0.08 0.06 0.08; visual mesh filename=../meshes/robot_arms/fer/visual/link3.dae
- link fer_link4: geometry collision box size=0.08 0.25 0.06; visual mesh filename=../meshes/robot_arms/fer/visual/link4.dae
- link fer_link5: geometry collision cylinder length=0.08 radius=0.035; visual mesh filename=../meshes/robot_arms/fer/visual/link5.dae
- link fer_link6: geometry collision box size=0.06 0.05 0.04; visual mesh filename=../meshes/robot_arms/fer/visual/link6.dae
- link fer_link7: geometry collision cylinder length=0.06 radius=0.03; visual mesh filename=../meshes/robot_arms/fer/visual/link7.dae
- link fer_rightfinger: geometry collision box size=0.008 0.012 0.035; visual mesh filename=../meshes/robot_ee/franka_hand_white/visual/finger.dae
