Commit message: Cleanup URDF bloatware

File: models/urdf/fer_drake.urdf (robot description, URDF)
Before this commit: robot fer, 14 links, 13 joints
Links:
- link fer_hand: geometry collision mesh filename=../meshes/robot_ee/franka_hand_white/collision/hand.obj; visual mesh filename=../meshes/robot_ee/franka_hand_white/visual/hand.dae
- link fer_leftfinger: geometry collision box size=0.01 0.01 0.04; visual mesh filename=../meshes/robot_ee/franka_hand_white/visual/finger.dae
- link fer_link0: geometry collision mesh filename=../meshes/robot_arms/fer/collision/link0.obj; visual mesh filename=../meshes/robot_arms/fer/visual/link0.dae
- link fer_link1: geometry collision mesh filename=../meshes/robot_arms/fer/collision/link1.obj; visual mesh filename=../meshes/robot_arms/fer/visual/link1.dae
- link fer_link2: geometry collision mesh filename=../meshes/robot_arms/fer/collision/link2.obj; visual mesh filename=../meshes/robot_arms/fer/visual/link2.dae
- link fer_link3: geometry collision mesh filename=../meshes/robot_arms/fer/collision/link3.obj; visual mesh filename=../meshes/robot_arms/fer/visual/link3.dae
- link fer_link4: geometry collision mesh filename=../meshes/robot_arms/fer/collision/link4.obj; visual mesh filename=../meshes/robot_arms/fer/visual/link4.dae
- link fer_link5: geometry collision mesh filename=../meshes/robot_arms/fer/collision/link5.obj; visual mesh filename=../meshes/robot_arms/fer/visual/link5.dae
- link fer_link6: geometry collision mesh filename=../meshes/robot_arms/fer/collision/link6.obj; visual mesh filename=../meshes/robot_arms/fer/visual/link6.dae
- link fer_link7: geometry collision mesh filename=../meshes/robot_arms/fer/collision/link7.obj; visual mesh filename=../meshes/robot_arms/fer/visual/link7.dae
- link fer_rightfinger: geometry collision box size=0.01 0.01 0.04; visual mesh filename=../meshes/robot_ee/franka_hand_white/visual/finger.dae
Joints:
- joint fer_finger_joint1: limit lower=0.0 upper=0.04 effort=100 velocity=0.2 -> lower=0.0 upper=0.04 effort=150 velocity=0.25
- joint fer_finger_joint2: limit lower=0.0 upper=0.04 effort=100 velocity=0.2 -> lower=0.0 upper=0.04 effort=150 velocity=0.25
